Commit message: second robot inclusion

File: iiwa_description/config/iiwa.config.xacro (robot description, xacro)
@@ -5,5 +5,7 @@
     <xacro:arg name="use_sim" default="false" />
     <xacro:arg name="use_fake_hardware" default="true" />
-    <xacro:arg name="prefix" default="" />
+    <!-- <xacro:arg name="prefix" default="" /> -->
+    <xacro:arg name="prefix_1" default="robot1_" />
+    <xacro:arg name="prefix_2" default="robot2_" />
     <xacro:arg name="robot_ip" default="192.170.10.2" />
     <xacro:arg name="robot_port" default="30200" />
@@ -29,10 +31,21 @@
     <xacro:property name="base_frame_file" value="$(arg base_frame_file)"/>
     <xacro:property name="base_frame" value="${xacro.load_yaml(base_frame_file)['base_frame']}"/>
-    <xacro:iiwa parent="world" prefix="$(arg prefix)">
+    <xacro:iiwa parent="world" prefix="$(arg prefix_1)">
+        <origin xyz="${base_frame['x']} ${base_frame['y']} ${base_frame['z']}"
+            rpy="${base_frame['roll']} ${base_frame['pitch']} ${base_frame['yaw']}" />
+    </xacro:iiwa>
+    <xacro:iiwa parent="world" prefix="$(arg prefix_2)">
         <origin xyz="${base_frame['x']} ${base_frame['y']} ${base_frame['z']}"
             rpy="${base_frame['roll']} ${base_frame['pitch']} ${base_frame['yaw']}" />
     </xacro:iiwa>
     <xacro:iiwa_r2c_hardware
-        name="iiwaRobot" prefix="$(arg prefix)"
+        name="iiwaRobot" prefix="$(arg prefix_1)"
+        robot_ip="$(arg robot_ip)" robot_port="$(arg robot_port)"
+        command_interface="$(arg command_interface)"
+        initial_positions_file="$(arg initial_positions_file)"
+        use_sim="$(arg use_sim)" use_fake_hardware="$(arg use_fake_hardware)"
+        />
+    <xacro:iiwa_r2c_hardware
+        name="iiwaRobot" prefix="$(arg prefix_2)"
         robot_ip="$(arg robot_ip)" robot_port="$(arg robot_port)"
         command_interface="$(arg command_interface)"
@@ -44,5 +57,11 @@
         controllers_file="$(arg controllers_file)"
         namespace="$(arg namespace)"
-        prefix="$(arg prefix)"
+        prefix="$(arg prefix_1)"
+        />
+    <xacro:iiwa_gazebo
+        runtime_config_package="$(arg runtime_config_package)"
+        controllers_file="$(arg controllers_file)"
+        namespace="$(arg namespace)"
+        prefix="$(arg prefix_2)"
         />
 </robot>

File: iiwa_description/urdf/iiwa.urdf.xacro (robot description, xacro)
@@ -3,280 +3,279 @@
   <!-- Contants -->
   <xacro:property name="PI" value="3.14159265359"/>
-  <xacro:macro name="iiwa" params="parent prefix *origin">
   <material name="gray">
     <color rgba="0.5 0.5 0.5 1.0"/>
   </material>
-<!-- Joint between the ${parent} and the added base -->
-<joint name="${prefix}iiwa_root_joint" type="fixed">
-  <origin xyz = "0 0 0.86" rpy = "${PI} 0 ${-PI/2}" />
-  <parent link="${parent}"/>
-  <child link="${prefix}iiwa_base"/>
-</joint>
-<!-- Added base -->
- <link name = "${prefix}iiwa_base">
+  <!-- Added base -->
+ <link name = "base">
+  <visual>
+    <origin xyz = "0 0 0" rpy = "0 0 0"/>
+    <geometry>
+      <mesh filename = "package://iiwa_description/meshes/flex_fellow_h800/flex_fellow_h800.dae"/>
+    </geometry>
+  </visual>
+  <collision>
+    <origin xyz = "0 0 0" rpy = "0 0 ${PI/2}"/>
+    <geometry>
+      <mesh filename = "package://iiwa_description/meshes/flex_fellow_h800/flex_fellow_h800.stl"/>
+    </geometry>
+  </collision>
+</link>
+      <!-- Added table plane-->
+<link name="table_plane">
       <visual>
-        <origin xyz = "0 0 0" rpy = "0 0 0"/>
-        <geometry>
-          <mesh filename = "package://iiwa_description/meshes/flex_fellow_h800/flex_fellow_h800.dae"/>
-        </geometry>
-      </visual>
-      <collision>
-        <origin xyz = "0 0 0" rpy = "0 0 ${PI/2}"/>
-        <geometry>
-          <mesh filename = "package://iiwa_description/meshes/flex_fellow_h800/flex_fellow_h800.stl"/>
-        </geometry>
-      </collision>
- </link>
-  <joint name="${prefix}iiwa_base_joint" type="fixed">
-      <origin rpy="${PI} 0 ${PI/2}" xyz="0.52 0 0"/>
-      <parent link="${prefix}iiwa_base"/>
-      <child link="${prefix}link_0"/>
-  </joint>
-  <link name="${prefix}link_0">
-      <visual>
+          <origin xyz = "0 0 0" rpy = "0 0 0"/>
+          <geometry>
+            <mesh filename = "package://iiwa_description/meshes/table_plane.stl" scale ="0.0001 0.0001 0.0001"/>
+          </geometry>
+        </visual>
+        <collision>
+          <origin xyz = "0 0 0" rpy = "0 0 0"/>
+          <geometry>
+            <mesh filename = "package://iiwa_description/meshes/table_plane.stl" scale ="0.0001 0.0001 0.0001"/>
+          </geometry>
+        </collision>
+      </link>
+      <!-- Joint Between the added base and the table-->
+<joint name="joint_a8" type="fixed">
+        <origin rpy="0 0 0" xyz="-0.3 0.50 0.10"/>
+        <parent link="base"/>
+        <child link="table_plane"/>
+        <axis xyz="0 0 0"/>
+    </joint>
+  <xacro:macro name="iiwa" params="parent prefix *origin">
+      <joint name="${prefix}iiwa_root_joint" type="fixed">
+        <xacro:insert_block name="origin" />
+        <parent link="${parent}"/>
+        <child link="base"/>
+      </joint>
+      <joint name="${prefix}iiwa_base_joint" type="fixed">
         <origin rpy="0.0 0 0" xyz="0 0 0"/>
-        <geometry>
-          <mesh filename="package://iiwa_description/meshes/lbr_iiwa_14_r820/visual/base_link.dae"/>
-        </geometry>
-      </visual>
-      <collision>
-        <origin rpy="0 0 0" xyz="0 0 0"/>
-        <geometry>
-          <mesh filename="package://iiwa_description/meshes/lbr_iiwa_14_r820/collision/base_link.stl"/>
-        </geometry>
-      </collision>
-      <inertial>
-        <origin xyz="-0.1 0 0.07" rpy="0 0 0"/>
-        <mass value="5"/>
-        <inertia ixx="0.05"  ixy="0"  ixz="0" iyy="0.06" iyz="0" izz="0.03" />
-      </inertial>
-  </link>
-  <link name="${prefix}link_1">
-      <visual>
-        <origin rpy="0 0 0" xyz="0 0 0"/>
-        <geometry>
-          <mesh filename="package://iiwa_description/meshes/lbr_iiwa_14_r820/visual/link_1.dae"/>
-        </geometry>
-      </visual>
-      <collision>
-        <origin rpy="0 0 0" xyz="0 0 0"/>
-        <geometry>
-          <mesh filename="package://iiwa_description/meshes/lbr_iiwa_14_r820/collision/link_1.stl"/>
-        </geometry>
-      </collision>
-      <inertial>
-        <origin xyz="0 -0.03 0.12" rpy="0 0 0"/>
-        <mass value="4"/>
-        <inertia ixx="0.1"  ixy="0"  ixz="0" iyy="0.09" iyz="0" izz="0.02" />
-      </inertial>
-  </link>
-  <link name="${prefix}link_2">
-      <visual>
-        <origin rpy="0 0 0" xyz="0 0 0"/>
-        <geometry>
-          <mesh filename="package://iiwa_description/meshes/lbr_iiwa_14_r820/visual/link_2.dae"/>
-        </geometry>
-      </visual>
-      <collision>
-        <origin rpy="0 0 0" xyz="0 0 0"/>
-        <geometry>
-          <mesh filename="package://iiwa_description/meshes/lbr_iiwa_14_r820/collision/link_2.stl"/>
-        </geometry>
-      </collision>
-      <inertial>
-        <origin xyz="0.0003 0.059 0.042" rpy="0 0 0"/>
-        <mass value="4"/>
-        <inertia ixx="0.05"  ixy="0"  ixz="0" iyy="0.018" iyz="0" izz="0.044" />
-      </inertial>
-  </link>
-  <link name="${prefix}link_3">
-      <visual>
-        <origin rpy="0 0 0" xyz="0 0 0"/>
-        <geometry>
-          <mesh filename="package://iiwa_description/meshes/lbr_iiwa_14_r820/visual/link_3.dae"/>
-        </geometry>
-      </visual>
-      <collision>
-        <origin rpy="0 0 0" xyz="0 0 0"/>
-        <geometry>
-          <mesh filename="package://iiwa_description/meshes/lbr_iiwa_14_r820/collision/link_3.stl"/>
-        </geometry>
-      </collision>
-      <inertial>
-        <origin xyz="0 0.03 0.13" rpy="0 0 0"/>
-        <mass value="3"/>
-        <inertia ixx="0.08"  ixy="0"  ixz="0" iyy="0.075" iyz="0" izz="0.01" />
-      </inertial>
-  </link>
-  <link name="${prefix}link_4">
-      <visual>
-        <origin rpy="0 0 0" xyz="0 0 0"/>
-        <geometry>
-          <mesh filename="package://iiwa_description/meshes/lbr_iiwa_14_r820/visual/link_4.dae"/>
-        </geometry>
-      </visual>
-      <collision>
-        <origin rpy="0 0 0" xyz="0 0 0"/>
-        <geometry>
-          <mesh filename="package://iiwa_description/meshes/lbr_iiwa_14_r820/collision/link_4.stl"/>
-        </geometry>
-      </collision>
-      <inertial>
-        <origin xyz="0 0.067 0.034" rpy="0 0 0"/>
-        <mass value="2.7"/>
-        <inertia ixx="0.03"  ixy="0"  ixz="0" iyy="0.01" iyz="0" izz="0.029" />
-      </inertial>
-  </link>
-  <link name="${prefix}link_5">
-      <visual>
-        <origin rpy="0 0 0" xyz="0 0 0"/>
-        <geometry>
-          <mesh filename="package://iiwa_description/meshes/lbr_iiwa_14_r820/visual/link_5.dae"/>
-        </geometry>
-      </visual>
-      <collision>
-        <origin rpy="0 0 0" xyz="0 0 0"/>
-        <geometry>
-          <mesh filename="package://iiwa_description/meshes/lbr_iiwa_14_r820/collision/link_5.stl"/>
-        </geometry>
-      </collision>
-      <inertial>
-        <origin xyz="0.0001 0.021 0.076" rpy="0 0 0"/>
-        <mass value="1.7"/>
-        <inertia ixx="0.02"  ixy="0"  ixz="0" iyy="0.018" iyz="0" izz="0.005" />
-      </inertial>
-  </link>
-  <link name="${prefix}link_6">
-      <visual>
-        <origin rpy="0 0 0" xyz="0 0 0"/>
-        <geometry>
-          <mesh filename="package://iiwa_description/meshes/lbr_iiwa_14_r820/visual/link_6.dae"/>
-        </geometry>
-      </visual>
-      <collision>
-        <origin rpy="0 0 0" xyz="0 0 0"/>
-        <geometry>
-          <mesh filename="package://iiwa_description/meshes/lbr_iiwa_14_r820/collision/link_6.stl"/>
-        </geometry>
-      </collision>
-      <inertial>
-        <origin xyz="0 0.0006 0.0004" rpy="0 0 0"/>
-        <mass value="1.8"/>
-        <inertia ixx="0.025"  ixy="0"  ixz="0" iyy="0.0136" iyz="0" izz="0.0247" />
-      </inertial>
-  </link>
-  <link name="${prefix}link_7">
-      <visual>
-        <origin rpy="0 0 0" xyz="0 0 0.07"/>
-        <material name="gray"/>
-        <geometry>
-          <mesh filename="package://iiwa_description/meshes/lbr_iiwa_14_r820/visual/link_7_2.stl" scale ="0.001 0.001 0.001"/>
-        </geometry>
-      </visual>
-      <collision>
-        <origin rpy="0 0 0" xyz="0 0 0.07"/>
-        <geometry>
-          <mesh filename="package://iiwa_description/meshes/lbr_iiwa_14_r820/collision/link_7_2.stl" scale ="0.001 0.001 0.001"/>
-        </geometry>
-      </collision>
-      <inertial>
-        <origin xyz="0 0 0.02" rpy="0 0 0"/>
-        <mass value="${0.3 / 0.308 * 0.44}"/> <!--this is for the MFT Pneumatisch flange-->
-        <inertia ixx="0.01"  ixy="0"  ixz="0" iyy="0.01" iyz="0" izz="0.01" />
-      </inertial>
-  </link>
-  <!-- Added Gripper Link-->
-  <link name="${prefix}tool0">
-    <visual>
-      <origin xyz = "0 0 0" rpy = "0 0 0"/>
-      <geometry>
-        <mesh filename = "package://iiwa_description/meshes/lbr_iiwa_14_r820/klt_gripper_iiwa_90_deg.stl" scale ="0.001 0.001 0.001"/>
-      </geometry>
-    </visual>
-    <collision>
-      <origin xyz = "0 0 0" rpy = "0 0 0"/>
-      <geometry>
-        <mesh filename = "package://iiwa_description/meshes/lbr_iiwa_14_r820/klt_gripper_iiwa_90_deg.stl" scale ="0.001 0.001 0.001"/>
-      </geometry>
-    </collision>
-  </link>
-  <!-- Added table plane-->
-  <link name="${prefix}table_plane">
-    <visual>
-      <origin xyz = "0 0 0" rpy = "0 0 0"/>
-      <geometry>
-        <mesh filename = "package://iiwa_description/meshes/table_plane.stl" scale ="0.0001 0.0001 0.0001"/>
-      </geometry>
-    </visual>
-    <collision>
-      <origin xyz = "0 0 0" rpy = "0 0 0"/>
-      <geometry>
-        <mesh filename = "package://iiwa_description/meshes/table_plane.stl" scale ="0.0001 0.0001 0.0001"/>
-      </geometry>
-    </collision>
-  </link>
-  <joint name="${prefix}joint_a1" type="revolute">
-      <origin rpy="0 0 0" xyz="0 0 0"/>
-      <parent link="${prefix}link_0"/>
-      <child link="${prefix}link_1"/>
-      <axis xyz="0 0 1"/>
-      <limit effort="320" lower="-2.9668" upper="2.9668" velocity="1.4834"/>
-  </joint>
-  <joint name="${prefix}joint_a2" type="revolute">
-      <origin rpy="0 ${PI/2} 0" xyz="-0.00043624 0 0.36"/>
-      <parent link="${prefix}link_1"/>
-      <child link="${prefix}link_2"/>
-      <axis xyz="0 1 0"/>
-      <limit effort="320" lower="-2.0942" upper="2.0942" velocity="1.4834"/>
-  </joint>
-  <joint name="${prefix}joint_a3" type="revolute">
-      <origin rpy="0 0 0" xyz="0 0 0"/>
-      <parent link="${prefix}link_2"/>
-      <child link="${prefix}link_3"/>
-      <axis xyz="0 0 1"/>
-      <limit effort="176" lower="-2.9668" upper="2.9668" velocity="1.7452"/>
-  </joint>
-  <joint name="${prefix}joint_a4" type="revolute">
-      <origin rpy="0 ${PI} 0" xyz="0.00043624 0 0.42"/>
-      <parent link="${prefix}link_3"/>
-      <child link="${prefix}link_4"/>
-      <axis xyz="0 -1 0"/>
-      <!-- <limit effort="176" lower="-2.0942" upper="2.0942" velocity="1.3089"/>  -->
-      <limit effort="176" lower="${-PI}" upper="${PI}" velocity="1.3089"/>
-  </joint>
-  <joint name="${prefix}joint_a5" type="revolute">
-      <origin rpy="0 0 0" xyz="0 0 0"/>
-      <parent link="${prefix}link_4"/>
-      <child link="${prefix}link_5"/>
-      <axis xyz="0 0 1"/>
-      <limit effort="110" lower="-2.9668" upper="2.9668" velocity="2.2688"/>
-  </joint>
-  <joint name="${prefix}joint_a6" type="revolute">
-      <origin rpy="0 0 0" xyz="0 0 0.4"/>
-      <parent link="${prefix}link_5"/>
-      <child link="${prefix}link_6"/>
-      <axis xyz="0 1 0"/>
-      <limit effort="40" lower="-2.0942" upper="2.0942" velocity="2.356"/>
-  </joint>
-  <joint name="${prefix}joint_a7" type="revolute">
-      <origin rpy="0 0 0" xyz="0 0 0"/>
-      <parent link="${prefix}link_6"/>
-      <child link="${prefix}link_7"/>
-      <axis xyz="0 0 1"/>
-      <limit effort="40" lower="-3.0541" upper="3.0541" velocity="2.356"/>
-  </joint>
-  <joint name="${prefix}joint_a7-tool0" type="fixed">
-      <origin rpy="0 ${PI/2} ${PI/2}" xyz="0 -0.06 0.205"/>
-      <parent link="${prefix}link_7"/>
-      <child link="${prefix}tool0"/>
-      <axis xyz="0 0 0"/>
-  </joint>
-  <!-- Joint Between the added base and the table-->
-  <joint name="${prefix}joint_a8" type="fixed">
-    <origin rpy="0 0 0" xyz="-0.3 0.50 0.10"/>
-    <parent link="${prefix}iiwa_base"/>
-    <child link="${prefix}table_plane"/>
-    <axis xyz="0 0 0"/>
-</joint>
+        <parent link="base"/>
+        <child link="${prefix}link_0"/>
+      </joint>
+      <link name="${prefix}link_0">
+          <visual>
+            <origin rpy="0.0 0 0" xyz="0 0 0"/>
+            <geometry>
+              <mesh filename="package://iiwa_description/meshes/lbr_iiwa_14_r820/visual/base_link.dae"/>
+            </geometry>
+          </visual>
+          <collision>
+            <origin rpy="0 0 0" xyz="0 0 0"/>
+            <geometry>
+              <mesh filename="package://iiwa_description/meshes/lbr_iiwa_14_r820/collision/base_link.stl"/>
+            </geometry>
+          </collision>
+          <inertial>
+            <origin xyz="-0.1 0 0.07" rpy="0 0 0"/>
+            <mass value="5"/>
+            <inertia ixx="0.05"  ixy="0"  ixz="0" iyy="0.06" iyz="0" izz="0.03" />
+          </inertial>
+      </link>
+      <link name="${prefix}link_1">
+          <visual>
+            <origin rpy="0 0 0" xyz="0 0 0"/>
+            <geometry>
+              <mesh filename="package://iiwa_description/meshes/lbr_iiwa_14_r820/visual/link_1.dae"/>
+            </geometry>
+          </visual>
+          <collision>
+            <origin rpy="0 0 0" xyz="0 0 0"/>
+            <geometry>
+              <mesh filename="package://iiwa_description/meshes/lbr_iiwa_14_r820/collision/link_1.stl"/>
+            </geometry>
+          </collision>
+          <inertial>
+            <origin xyz="0 -0.03 0.12" rpy="0 0 0"/>
+            <mass value="4"/>
+            <inertia ixx="0.1"  ixy="0"  ixz="0" iyy="0.09" iyz="0" izz="0.02" />
+          </inertial>
+      </link>
+      <link name="${prefix}link_2">
+          <visual>
+            <origin rpy="0 0 0" xyz="0 0 0"/>
+            <geometry>
+              <mesh filename="package://iiwa_description/meshes/lbr_iiwa_14_r820/visual/link_2.dae"/>
+            </geometry>
+          </visual>
+          <collision>
+            <origin rpy="0 0 0" xyz="0 0 0"/>
+            <geometry>
+              <mesh filename="package://iiwa_description/meshes/lbr_iiwa_14_r820/collision/link_2.stl"/>
+            </geometry>
+          </collision>
+          <inertial>
+            <origin xyz="0.0003 0.059 0.042" rpy="0 0 0"/>
+            <mass value="4"/>
+            <inertia ixx="0.05"  ixy="0"  ixz="0" iyy="0.018" iyz="0" izz="0.044" />
+          </inertial>
+      </link>
+      <link name="${prefix}link_3">
+          <visual>
+            <origin rpy="0 0 0" xyz="0 0 0"/>
+            <geometry>
+              <mesh filename="package://iiwa_description/meshes/lbr_iiwa_14_r820/visual/link_3.dae"/>
+            </geometry>
+          </visual>
+          <collision>
+            <origin rpy="0 0 0" xyz="0 0 0"/>
+            <geometry>
+              <mesh filename="package://iiwa_description/meshes/lbr_iiwa_14_r820/collision/link_3.stl"/>
+            </geometry>
+          </collision>
+          <inertial>
+            <origin xyz="0 0.03 0.13" rpy="0 0 0"/>
+            <mass value="3"/>
+            <inertia ixx="0.08"  ixy="0"  ixz="0" iyy="0.075" iyz="0" izz="0.01" />
+          </inertial>
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