Commit message: with controllers loaded

File: iiwa_description/ros2_control/iiwa.r2c_hardware.xacro (robot description, xacro)
@@ -2,148 +2,296 @@
 <robot xmlns:xacro="http://www.ros.org/wiki/xacro">
     <xacro:macro name="iiwa_r2c_hardware" params="name prefix command_interface robot_ip robot_port initial_positions_file use_sim:=^|false use_fake_hardware:=^|true">
-        <xacro:property name="initial_positions" value="${xacro.load_yaml(initial_positions_file)['initial_positions']}"/>
-        <ros2_control name="${name}" type="system">
-            <xacro:if value="$(arg use_sim)">
-                <hardware>
-                    <plugin>gazebo_ros2_control/GazeboSystem</plugin>
-                </hardware>
-            </xacro:if>
-            <xacro:unless value="$(arg use_sim)">
-                <hardware>
-                <xacro:if value="${use_fake_hardware}">
-                    <plugin>fake_components/GenericSystem</plugin>
-                        <param name="state_following_offset">0.0</param>
+        <xacro:if value = "${prefix == 'robot1_'}">
+            <xacro:property name="initial_positions" value="${xacro.load_yaml(initial_positions_file)['initial_positions']}"/>
+            <ros2_control name="${prefix}${name}" type="system">
+                <xacro:if value="$(arg use_sim)">
+                    <hardware>
+                        <plugin>gazebo_ros2_control/GazeboSystem</plugin>
+                    </hardware>
                 </xacro:if>
-                <xacro:unless value="${use_fake_hardware}">
-                    <plugin>iiwa_hardware/IiwaFRIHardwareInterface</plugin>
-                    <param name="robot_ip">${robot_ip}</param>
-                    <param name="robot_port">${robot_port}</param>
-                    <param name="velocity_filter_cutoff_freq">40</param>
-                    <param name="torque_filter_cutoff_freq">40</param>
+                <xacro:unless value="$(arg use_sim)">
+                    <hardware>
+                        <xacro:if value="${use_fake_hardware}">
+                            <plugin>fake_components/GenericSystem</plugin>
+                            <param name="state_following_offset">0.0</param>
+                        </xacro:if>
+                        <xacro:unless value="${use_fake_hardware}">
+                            <plugin>iiwa_hardware/IiwaFRIHardwareInterface</plugin>
+                            <param name="robot_ip">${robot_ip}</param>
+                            <param name="robot_port">${robot_port}</param>
+                            <param name="velocity_filter_cutoff_freq">40</param>
+                            <param name="torque_filter_cutoff_freq">40</param>
+                        </xacro:unless>
+                    </hardware>
                 </xacro:unless>
-                </hardware>
-            </xacro:unless>
-            <joint name="${prefix}joint_a1">
-                <command_interface name="${command_interface}" />
-                    <xacro:if value="${command_interface == 'position'}">
-                        <param name="min">-2.96</param>
-                        <param name="max">2.96</param>
-                    </xacro:if>
-                <state_interface name="position">
-                    <param name="initial_value">${initial_positions['joint_a1']}</param>
-                </state_interface>
-                <state_interface name="velocity">
-                    <param name="initial_value">0.0</param>
-                </state_interface>
-                <state_interface name="effort">
-                    <param name="initial_value">0.0</param>
-                </state_interface>
-            </joint>
-            <joint name="${prefix}joint_a2">
-                <command_interface name="${command_interface}" />
-                    <xacro:if value="${command_interface == 'position'}">
-                        <param name="min">-2.09</param>
-                        <param name="max">2.09</param>
-                    </xacro:if>
-                <state_interface name="position">
-                    <param name="initial_value">${initial_positions['joint_a2']}</param>
-                </state_interface>
-                <state_interface name="velocity">
-                    <param name="initial_value">0.0</param>
-                </state_interface>
-                <state_interface name="effort">
-                    <param name="initial_value">0.0</param>
-                </state_interface>
-            </joint>
-            <joint name="${prefix}joint_a3">
-                <command_interface name="${command_interface}" />
-                    <xacro:if value="${command_interface == 'position'}">
-                        <param name="min">-2.96</param>
-                        <param name="max">2.96</param>
-                    </xacro:if>
-                <state_interface name="position">
-                    <param name="initial_value">${initial_positions['joint_a3']}</param>
-                </state_interface>
-                <state_interface name="velocity">
-                    <param name="initial_value">0.0</param>
-                </state_interface>
-                <state_interface name="effort">
-                    <param name="initial_value">0.0</param>
-                </state_interface>
-            </joint>
-            <joint name="${prefix}joint_a4">
-                <command_interface name="${command_interface}" />
-                    <xacro:if value="${command_interface == 'position'}">
-                        <param name="min">-2.09</param>
-                        <param name="max">2.09</param>
-                    </xacro:if>
-                <state_interface name="position">
-                    <param name="initial_value">${initial_positions['joint_a4']}</param>
-                </state_interface>
-                <state_interface name="velocity">
-                    <param name="initial_value">0.0</param>
-                </state_interface>
-                <state_interface name="effort">
-                    <param name="initial_value">0.0</param>
-                </state_interface>
-            </joint>
-            <joint name="${prefix}joint_a5">
-                <command_interface name="${command_interface}" />
-                    <xacro:if value="${command_interface == 'position'}">
-                        <param name="min">-2.96</param>
-                        <param name="max">2.96</param>
-                    </xacro:if>
-                <state_interface name="position">
-                    <param name="initial_value">${initial_positions['joint_a5']}</param>
-                </state_interface>
-                <state_interface name="velocity">
-                    <param name="initial_value">0.0</param>
-                </state_interface>
-                <state_interface name="effort">
-                    <param name="initial_value">0.0</param>
-                </state_interface>
-            </joint>
-            <joint name="${prefix}joint_a6">
-                <command_interface name="${command_interface}" />
-                    <xacro:if value="${command_interface == 'position'}">
-                        <param name="min">-2.09</param>
-                        <param name="max">2.09</param>
-                    </xacro:if>
-                <state_interface name="position">
-                    <param name="initial_value">${initial_positions['joint_a6']}</param>
-                </state_interface>
-                <state_interface name="velocity">
-                    <param name="initial_value">0.0</param>
-                </state_interface>
-                <state_interface name="effort">
-                    <param name="initial_value">0.0</param>
-                </state_interface>
-            </joint>
-            <joint name="${prefix}joint_a7">
-                <command_interface name="${command_interface}" />
+                <joint name="${prefix}joint_a1">
+                    <command_interface name="${command_interface}" />
+                    <xacro:if value="${command_interface == 'position'}">
+                        <param name="min">-2.96</param>
+                        <param name="max">2.96</param>
+                    </xacro:if>
+                    <state_interface name="position">
+                        <param name="initial_value">${initial_positions['robot1_joint_a1']}</param>
+                    </state_interface>
+                    <state_interface name="velocity">
+                        <param name="initial_value">0.0</param>
+                    </state_interface>
+                    <state_interface name="effort">
+                        <param name="initial_value">0.0</param>
+                    </state_interface>
+                </joint>
+                <joint name="${prefix}joint_a2">
+                    <command_interface name="${command_interface}" />
+                    <xacro:if value="${command_interface == 'position'}">
+                        <param name="min">-2.09</param>
+                        <param name="max">2.09</param>
+                    </xacro:if>
+                    <state_interface name="position">
+                        <param name="initial_value">${initial_positions['robot1_joint_a2']}</param>
+                    </state_interface>
+                    <state_interface name="velocity">
+                        <param name="initial_value">0.0</param>
+                    </state_interface>
+                    <state_interface name="effort">
+                        <param name="initial_value">0.0</param>
+                    </state_interface>
+                </joint>
+                <joint name="${prefix}joint_a3">
+                    <command_interface name="${command_interface}" />
+                    <xacro:if value="${command_interface == 'position'}">
+                        <param name="min">-2.96</param>
+                        <param name="max">2.96</param>
+                    </xacro:if>
+                    <state_interface name="position">
+                        <param name="initial_value">${initial_positions['robot1_joint_a3']}</param>
+                    </state_interface>
+                    <state_interface name="velocity">
+                        <param name="initial_value">0.0</param>
+                    </state_interface>
+                    <state_interface name="effort">
+                        <param name="initial_value">0.0</param>
+                    </state_interface>
+                </joint>
+                <joint name="${prefix}joint_a4">
+                    <command_interface name="${command_interface}" />
+                    <xacro:if value="${command_interface == 'position'}">
+                        <param name="min">-2.09</param>
+                        <param name="max">2.09</param>
+                    </xacro:if>
+                    <state_interface name="position">
+                        <param name="initial_value">${initial_positions['robot1_joint_a4']}</param>
+                    </state_interface>
+                    <state_interface name="velocity">
+                        <param name="initial_value">0.0</param>
+                    </state_interface>
+                    <state_interface name="effort">
+                        <param name="initial_value">0.0</param>
+                    </state_interface>
+                </joint>
+                <joint name="${prefix}joint_a5">
+                    <command_interface name="${command_interface}" />
+                    <xacro:if value="${command_interface == 'position'}">
+                        <param name="min">-2.96</param>
+                        <param name="max">2.96</param>
+                    </xacro:if>
+                    <state_interface name="position">
+                        <param name="initial_value">${initial_positions['robot1_joint_a5']}</param>
+                    </state_interface>
+                    <state_interface name="velocity">
+                        <param name="initial_value">0.0</param>
+                    </state_interface>
+                    <state_interface name="effort">
+                        <param name="initial_value">0.0</param>
+                    </state_interface>
+                </joint>
+                <joint name="${prefix}joint_a6">
+                    <command_interface name="${command_interface}" />
+                    <xacro:if value="${command_interface == 'position'}">
+                        <param name="min">-2.09</param>
+                        <param name="max">2.09</param>
+                    </xacro:if>
+                    <state_interface name="position">
+                        <param name="initial_value">${initial_positions['robot1_joint_a6']}</param>
+                    </state_interface>
+                    <state_interface name="velocity">
+                        <param name="initial_value">0.0</param>
+                    </state_interface>
+                    <state_interface name="effort">
+                        <param name="initial_value">0.0</param>
+                    </state_interface>
+                </joint>
+                <joint name="${prefix}joint_a7">
+                    <command_interface name="${command_interface}" />
                     <xacro:if value="${command_interface == 'position'}">
                         <param name="min">-3.05</param>
                         <param name="max">3.05</param>
                     </xacro:if>
-                <state_interface name="position">
-                    <param name="initial_value">${initial_positions['joint_a7']}</param>
-                </state_interface>
-                <state_interface name="velocity">
-                    <param name="initial_value">0.0</param>
-                </state_interface>
-                <state_interface name="effort">
-                    <param name="initial_value">0.0</param>
-                </state_interface>
-            </joint>
-            <sensor name="${prefix}external_torque_sensor">
-                <state_interface name="external_torque.joint_a1"/>
-                <state_interface name="external_torque.joint_a2"/>
-                <state_interface name="external_torque.joint_a3"/>
-                <state_interface name="external_torque.joint_a4"/>
-                <state_interface name="external_torque.joint_a5"/>
-                <state_interface name="external_torque.joint_a6"/>
-                <state_interface name="external_torque.joint_a7"/>
-            </sensor>
-        </ros2_control>
+                    <state_interface name="position">
+                        <param name="initial_value">${initial_positions['robot1_joint_a7']}</param>
+                    </state_interface>
+                    <state_interface name="velocity">
+                        <param name="initial_value">0.0</param>
+                    </state_interface>
+                    <state_interface name="effort">
+                        <param name="initial_value">0.0</param>
+                    </state_interface>
+                </joint>
+                <sensor name="${prefix}external_torque_sensor">
+                    <state_interface name="external_torque.{prefix}joint_a1"/>
+                    <state_interface name="external_torque.{prefix}joint_a2"/>
+                    <state_interface name="external_torque.{prefix}joint_a3"/>
+                    <state_interface name="external_torque.{prefix}joint_a4"/>
+                    <state_interface name="external_torque.{prefix}joint_a5"/>
+                    <state_interface name="external_torque.{prefix}joint_a6"/>
+                    <state_interface name="external_torque.{prefix}joint_a7"/>
+                </sensor>
+            </ros2_control>
+        </xacro:if>
+        <xacro:if value = "${prefix == 'robot2_'}">
+            <xacro:property name="initial_positions" value="${xacro.load_yaml(initial_positions_file)['initial_positions']}"/>
+            <ros2_control name="${prefix}${name}" type="system">
+                <xacro:if value="$(arg use_sim)">
+                    <hardware>
+                        <plugin>gazebo_ros2_control/GazeboSystem</plugin>
+                    </hardware>
+                </xacro:if>
+                <xacro:unless value="$(arg use_sim)">
+                    <hardware>
+                        <xacro:if value="${use_fake_hardware}">
+                            <plugin>fake_components/GenericSystem</plugin>
+                            <param name="state_following_offset">0.0</param>
+                        </xacro:if>
+                        <xacro:unless value="${use_fake_hardware}">
+                            <plugin>iiwa_hardware/IiwaFRIHardwareInterface</plugin>
+                            <param name="robot_ip">${robot_ip}</param>
+                            <param name="robot_port">${robot_port}</param>
+                            <param name="velocity_filter_cutoff_freq">40</param>
+                            <param name="torque_filter_cutoff_freq">40</param>
+                        </xacro:unless>
+                    </hardware>
+                </xacro:unless>
+                <joint name="${prefix}joint_a1">
+                    <command_interface name="${command_interface}" />
+                    <xacro:if value="${command_interface == 'position'}">
+                        <param name="min">-2.96</param>
+                        <param name="max">2.96</param>
+                    </xacro:if>
+                    <state_interface name="position">
+                        <param name="initial_value">${initial_positions['robot2_joint_a1']}</param>
+                    </state_interface>
+                    <state_interface name="velocity">
+                        <param name="initial_value">0.0</param>
+                    </state_interface>
+                    <state_interface name="effort">
+                        <param name="initial_value">0.0</param>
+                    </state_interface>
+                </joint>
+                <joint name="${prefix}joint_a2">
+                    <command_interface name="${command_interface}" />
+                    <xacro:if value="${command_interface == 'position'}">
+                        <param name="min">-2.09</param>
+                        <param name="max">2.09</param>
+                    </xacro:if>
+                    <state_interface name="position">
+                        <param name="initial_value">${initial_positions['robot2_joint_a2']}</param>
+                    </state_interface>
+                    <state_interface name="velocity">
+                        <param name="initial_value">0.0</param>
+                    </state_interface>
+                    <state_interface name="effort">
+                        <param name="initial_value">0.0</param>
+                    </state_interface>
+                </joint>
+                <joint name="${prefix}joint_a3">
+                    <command_interface name="${command_interface}" />
+                    <xacro:if value="${command_interface == 'position'}">
+                        <param name="min">-2.96</param>
+                        <param name="max">2.96</param>
+                    </xacro:if>
+                    <state_interface name="position">
+                        <param name="initial_value">${initial_positions['robot2_joint_a3']}</param>
+                    </state_interface>
+                    <state_interface name="velocity">
+                        <param name="initial_value">0.0</param>
+                    </state_interface>
+                    <state_interface name="effort">
+                        <param name="initial_value">0.0</param>
+                    </state_interface>
+                </joint>
+                <joint name="${prefix}joint_a4">
+                    <command_interface name="${command_interface}" />
+                    <xacro:if value="${command_interface == 'position'}">
+                        <param name="min">-2.09</param>
+                        <param name="max">2.09</param>
+                    </xacro:if>
+                    <state_interface name="position">
+                        <param name="initial_value">${initial_positions['robot2_joint_a4']}</param>
+                    </state_interface>
+                    <state_interface name="velocity">
+                        <param name="initial_value">0.0</param>
+                    </state_interface>
+                    <state_interface name="effort">
+                        <param name="initial_value">0.0</param>
+                    </state_interface>
+                </joint>
+                <joint name="${prefix}joint_a5">
+                    <command_interface name="${command_interface}" />
+                    <xacro:if value="${command_interface == 'position'}">
+                        <param name="min">-2.96</param>
+                        <param name="max">2.96</param>
+                    </xacro:if>
+                    <state_interface name="position">
+                        <param name="initial_value">${initial_positions['robot2_joint_a5']}</param>
+                    </state_interface>
+                    <state_interface name="velocity">
+                        <param name="initial_value">0.0</param>
+                    </state_interface>
+                    <state_interface name="effort">
+                        <param name="initial_value">0.0</param>
+                    </state_interface>
+                </joint>
+                <joint name="${prefix}joint_a6">
+                    <command_interface name="${command_interface}" />
+                    <xacro:if value="${command_interface == 'position'}">
+                        <param name="min">-2.09</param>
+                        <param name="max">2.09</param>
+                    </xacro:if>
+                    <state_interface name="position">
+                        <param name="initial_value">${initial_positions['robot2_joint_a6']}</param>
+                    </state_interface>
+                    <state_interface name="velocity">
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
File: iiwa_description/srdf/iiwa.srdf.xacro (robot description, xacro)
@@ -2,8 +2,10 @@
 <robot xmlns:xacro="http://wiki.ros.org/xacro" name="$(arg name)">
   <xacro:arg name="name" default="iiwa"/>
-  <xacro:arg name="prefix" default="" />
+  <xacro:arg name="prefix_1" default="prefix_1" />
+  <xacro:arg name="prefix_2" default="prefix_2" />
   <xacro:arg name="description_package" default="iiwa_description" />
   <xacro:property name="description_package" value="$(arg description_package)"/>
   <xacro:include filename="$(find ${description_package})/srdf/iiwa_macro.srdf.xacro"/>
-  <xacro:iiwa_srdf name="$(arg name)" prefix="$(arg prefix)"/>
+  <xacro:iiwa_srdf name="$(arg name)" prefix="$(arg prefix_1)"/>
+  <xacro:iiwa_srdf name="$(arg name)" prefix="$(arg prefix_2)"/>
 </robot>
