Commit message: with controllers loaded

File: iiwa_description/srdf/iiwa_macro.srdf.xacro (robot description, xacro)
@@ -3,5 +3,5 @@
   <xacro:macro name="iiwa_srdf" params="name prefix">
      <group name="${prefix}${name}_arm">
-        <chain base_link="${prefix}iiwa_base" tip_link="${prefix}tool0" />
+        <chain base_link="iiwa_base" tip_link="${prefix}tool0" />
     </group>
     <group_state name="ready" group="${prefix}${name}_arm">
@@ -14,9 +14,9 @@
         <joint name="${prefix}joint_a7" value="0.785"/>
     </group_state>
-    <virtual_joint child_link="${prefix}iiwa_base" name="virtual_joint" parent_frame="world" type="floating"/>
-    <disable_collisions link1="${prefix}iiwa_base" link2="${prefix}link_0" reason="Adjacent" />
-    <disable_collisions link1="${prefix}iiwa_base" link2="${prefix}link_1" reason="Never" />
-    <disable_collisions link1="${prefix}iiwa_base" link2="${prefix}link_2" reason="Never" />
-    <disable_collisions link1="${prefix}iiwa_base" link2="${prefix}link_3" reason="Never" />
+    <virtual_joint child_link="iiwa_base" name="virtual_joint" parent_frame="world" type="floating"/>
+    <disable_collisions link1="iiwa_base" link2="${prefix}link_0" reason="Adjacent" />
+    <disable_collisions link1="iiwa_base" link2="${prefix}link_1" reason="Never" />
+    <disable_collisions link1="iiwa_base" link2="${prefix}link_2" reason="Never" />
+    <disable_collisions link1="iiwa_base" link2="${prefix}link_3" reason="Never" />
     <disable_collisions link1="${prefix}link_0" link2="${prefix}link_1" reason="Adjacent" />
     <disable_collisions link1="${prefix}link_0" link2="${prefix}link_2" reason="Never" />
@@ -45,4 +45,5 @@
     <disable_collisions link1="${prefix}link_6" link2="${prefix}link_7" reason="Adjacent" />
     <disable_collisions link1="${prefix}link_7" link2="${prefix}tool0" reason="Adjacent" />
+    <disable_collisions link1="${prefix}tool0" link2 = "${prefix}tcp" reason="Adjacent"/>
   </xacro:macro>
 </robot>

File: iiwa_description/urdf/iiwa.urdf.xacro (robot description, xacro)
@@ -6,6 +6,9 @@
     <color rgba="0.5 0.5 0.5 1.0"/>
   </material>
+  <material name="blue">
+    <color rgba="0.0 0.0 1.0 1.0"/>
+  </material>
   <!-- Added base -->
-  <link name = "base">
+  <link name = "iiwa_base" type="fixed">
     <visual>
       <origin xyz = "0 0 0" rpy = "0 0 0"/>
@@ -38,6 +41,6 @@
   <!-- Joint Between the added base and the table-->
   <joint name="joint_a8" type="fixed">
-    <origin rpy="0 0 0" xyz="-0.3 0.50 0.10"/>
-    <parent link="base"/>
+    <origin rpy="0 0 0" xyz="-0.3 0.31 0.10"/>
+    <parent link="iiwa_base"/>
     <child link="table_plane"/>
   </joint>
@@ -46,9 +49,9 @@
       <origin xyz="-0.25 0.0 0.90" rpy="${PI} 0.0 0.0"/>
       <parent link="${parent}"/>
-      <child link="base"/>
+      <child link="iiwa_base"/>
     </joint>
     <joint name="${prefix}iiwa_base_joint" type="fixed">
       <xacro:insert_block name="origin" />
-      <parent link="base"/>
+      <parent link="iiwa_base"/>
       <child link="${prefix}link_0"/>
     </joint>
@@ -219,4 +222,20 @@
         <geometry>
           <mesh filename = "package://iiwa_description/meshes/lbr_iiwa_14_r820/klt_gripper_iiwa_90_deg.stl" scale ="0.001 0.001 0.001"/>
+        </geometry>
+      </collision>
+    </link>
+    <!-- TCP Link -->
+    <link name = "${prefix}tcp">
+      <visual>
+        <origin xyz = "0 0 0" rpy = "0 0 0"/>
+        <material name="blue"/>
+        <geometry>
+          <sphere radius = "0.01"/>
+        </geometry>
+      </visual>
+      <collision>
+        <origin xyz = "0 0 0" rpy = "0 0 0"/>
+        <geometry>
+          <sphere radius = "0.01"/>
         </geometry>
       </collision>
@@ -277,4 +296,9 @@
       <axis xyz="0 0 0"/>
     </joint>
+    <joint name="${prefix}tcp_joint" type="fixed">
+      <origin xyz="-0.05 0.0 0.0" rpy="0.0 ${PI} 0"/>
+      <parent link="${prefix}tool0"/>
+      <child link="${prefix}tcp"/>
+    </joint>
   </xacro:macro>
 </robot>
