Commit message: update un the urdf file so that the robots spawns with tool away from the table

File: iiwa_description/config/iiwa_robots.urdf (robot description, URDF)
Before this commit: robot iiwa, 23 links, 23 joints
Joints:
- joint robot1_joint_a2: axis 0 1 0 -> 0 -1 0; limit lower=-2.0942 upper=2.0942 effort=320 velocity=1.4834 -> lower=0 upper=4.1888 effort=320 velocity=1.4834; origin xyz=-0.00043624 0 0.36 rpy=0 -1.0471975511966667 0 -> xyz=-0.00043624 0 0.36 rpy=0 1.5708 0
- joint robot1_joint_a4: origin xyz=0.00043624 0 0.42 rpy=0 -1.570796326795 0 -> xyz=0.00043624 0 0.42 rpy=0 0 0
- joint robot2_joint_a2: limit lower=-2.0942 upper=2.0942 effort=320 velocity=1.4834 -> lower=0 upper=4.1888 effort=320 velocity=1.4834; origin xyz=-0.00043624 0 0.36 rpy=0 1.0471975511966667 0 -> xyz=-0.00043624 0 0.36 rpy=0 -1.5708 0
- joint robot2_joint_a4: origin xyz=0.00043624 0 0.42 rpy=0 1.570796326795 0 -> xyz=0.00043624 0 0.42 rpy=0 0 0

Commit message: collision issue solved

File: iiwa_description/config/iiwa_robots.urdf (robot description, URDF)
Before this commit: robot iiwa, 23 links, 23 joints
Joints:
- removed joint robot1_iiwa_root_joint
- removed joint robot2_iiwa_root_joint
- added joint iiwa_root_joint: type fixed, parent world, child iiwa_base, origin xyz=-0.25 0.0 0.90 rpy=3.14159265359 0.0 0.0
- joint robot1_joint_a2: axis 0 -1 0 -> 0 1 0; limit lower=0 upper=4.1888 effort=320 velocity=1.4834 -> lower=-2.0942 upper=2.0942 effort=320 velocity=1.4834; origin xyz=-0.00043624 0 0.36 rpy=0 1.5708 0 -> xyz=-0.00043624 0 0.36 rpy=0 -1.0471975511966667 0
- joint robot1_joint_a4: origin xyz=0.00043624 0 0.42 rpy=0 0 0 -> xyz=0.00043624 0 0.42 rpy=0 -1.570796326795 0
- joint robot2_joint_a2: limit lower=0 upper=4.1888 effort=320 velocity=1.4834 -> lower=-2.0942 upper=2.0942 effort=320 velocity=1.4834; origin xyz=-0.00043624 0 0.36 rpy=0 -1.5708 0 -> xyz=-0.00043624 0 0.36 rpy=0 1.0471975511966667 0
- joint robot2_joint_a4: origin xyz=0.00043624 0 0.42 rpy=0 0 0 -> xyz=0.00043624 0 0.42 rpy=0 1.570796326795 0

File: iiwa_description/urdf/iiwa.urdf.xacro (robot description, xacro)
@@ -24,4 +24,9 @@
     </collision>
   </link>
+  <joint name="iiwa_root_joint" type="fixed">
+    <origin xyz="-0.25 0.0 0.90" rpy="${PI} 0.0 ${PI}"/>
+    <parent link="world"/>
+    <child link="iiwa_base"/>
+  </joint>
   <!-- Added table plane-->
   <link name="table_plane">
@@ -46,9 +51,4 @@
   </joint>
   <xacro:macro name="iiwa" params="parent prefix pose_dir *origin">
-    <joint name="${prefix}iiwa_root_joint" type="fixed">
-      <origin xyz="-0.25 0.0 0.90" rpy="${PI} 0.0 0.0"/>
-      <parent link="${parent}"/>
-      <child link="iiwa_base"/>
-    </joint>
     <joint name="${prefix}iiwa_base_joint" type="fixed">
       <xacro:insert_block name="origin" />
