Commit message: added table_plane base and endeffector to urdf

File: iiwa_description/urdf/iiwa.urdf.xacro (robot description, xacro)
@@ -1,16 +1,33 @@
 <?xml version="1.0"?>
 <robot xmlns:xacro="http://www.ros.org/wiki/xacro">
+  <!-- Contants -->
+  <xacro:property name="PI" value="3.14159265359"/>
   <xacro:macro name="iiwa" params="parent prefix *origin">
   <material name="gray">
     <color rgba="0.5 0.5 0.5 1.0"/>
   </material>
-  <link name="${prefix}iiwa_base" type="fixed"/>
+<!-- Joint between the ${parent} and the added base -->
   <joint name="${prefix}iiwa_root_joint" type="fixed">
-      <xacro:insert_block name="origin" />
+      <origin xyz = "0 0 0.86" rpy = "${PI} 0 ${-PI/2}" />
       <parent link="${parent}"/>
       <child link="${prefix}iiwa_base"/>
   </joint>
+<!-- Added base -->
+ <link name = "${prefix}iiwa_base">
+      <visual>
+        <origin xyz = "0 0 0" rpy = "0 0 0"/>
+        <geometry>
+          <mesh filename = "package://iiwa_description/meshes/flex_fellow_h800/flex_fellow_h800.dae"/>
+        </geometry>
+      </visual>
+      <collision>
+        <origin xyz = "0 0 0" rpy = "0 0 0"/>
+        <geometry>
+          <mesh filename = "package://iiwa_description/meshes/flex_fellow_h800/flex_fellow_h800.stl"/>
+        </geometry>
+      </collision>
+ </link>
   <joint name="${prefix}iiwa_base_joint" type="fixed">
-      <origin rpy="0.0 0 0" xyz="0 0 0"/>
+      <origin rpy="${PI} 0 ${-PI/2}" xyz="0 0 0"/>
       <parent link="${prefix}iiwa_base"/>
       <child link="${prefix}link_0"/>
@@ -169,5 +186,34 @@
       </inertial>
   </link>
-  <link name="${prefix}tool0"/>
+  <!-- Added Gripper Link-->
+  <link name="${prefix}tool0">
+    <visual>
+      <origin xyz = "0 0 0" rpy = "0 0 0"/>
+      <geometry>
+        <mesh filename = "package://iiwa_description/meshes/lbr_iiwa_14_r820/klt_gripper_iiwa_90_deg.stl" scale ="0.001 0.001 0.001"/>
+      </geometry>
+    </visual>
+    <collision>
+      <origin xyz = "0 0 0" rpy = "0 0 0"/>
+      <geometry>
+        <mesh filename = "package://iiwa_description/meshes/lbr_iiwa_14_r820/klt_gripper_iiwa_90_deg.stl" scale ="0.001 0.001 0.001"/>
+      </geometry>
+    </collision>
+  </link>
+  <!-- Added table plane-->
+  <link name="${prefix}table_plane">
+    <visual>
+      <origin xyz = "0 0 0" rpy = "0 0 0"/>
+      <geometry>
+        <mesh filename = "package://iiwa_description/meshes/table_plane.stl" scale ="0.0001 0.0001 0.0001"/>
+      </geometry>
+    </visual>
+    <collision>
+      <origin xyz = "0 0 0" rpy = "0 0 0"/>
+      <geometry>
+        <mesh filename = "package://iiwa_description/meshes/table_plane.stl" scale ="0.0001 0.0001 0.0001"/>
+      </geometry>
+    </collision>
+  </link>
   <joint name="${prefix}joint_a1" type="revolute">
       <origin rpy="0 0 0" xyz="0 0 0"/>
@@ -220,9 +266,16 @@
   </joint>
   <joint name="${prefix}joint_a7-tool0" type="fixed">
-      <origin rpy="0 0 0" xyz="0 0 0.154"/>
+      <origin rpy="0 ${PI/2} ${PI/2}" xyz="0 -0.06 0.205"/>
       <parent link="${prefix}link_7"/>
       <child link="${prefix}tool0"/>
       <axis xyz="0 0 0"/>
   </joint>
+  <!-- Joint Between the added base and the table-->
+  <joint name="${prefix}joint_a8" type="fixed">
+    <origin rpy="0 0 0" xyz="-0.3 0.50 0.10"/>
+    <parent link="${prefix}iiwa_base"/>
+    <child link="${prefix}table_plane"/>
+    <axis xyz="0 0 0"/>
+</joint>
   </xacro:macro>
 </robot>

Commit message: moved the robot to the left side of the base and adjusted the pose to match what in the screenshot

File: iiwa_description/urdf/iiwa.urdf.xacro (robot description, xacro)
@@ -29,5 +29,5 @@
  </link>
   <joint name="${prefix}iiwa_base_joint" type="fixed">
-      <origin rpy="${PI} 0 ${-PI/2}" xyz="0 0 0"/>
+      <origin rpy="${PI} 0 ${PI/2}" xyz="0.52 0 0"/>
       <parent link="${prefix}iiwa_base"/>
       <child link="${prefix}link_0"/>
@@ -224,5 +224,5 @@
   </joint>
   <joint name="${prefix}joint_a2" type="revolute">
-      <origin rpy="0 0 0" xyz="-0.00043624 0 0.36"/>
+      <origin rpy="0 ${PI/2} 0" xyz="-0.00043624 0 0.36"/>
       <parent link="${prefix}link_1"/>
       <child link="${prefix}link_2"/>
@@ -238,5 +238,5 @@
   </joint>
   <joint name="${prefix}joint_a4" type="revolute">
-      <origin rpy="0 0 0" xyz="0.00043624 0 0.42"/>
+      <origin rpy="0 ${PI} 0" xyz="0.00043624 0 0.42"/>
       <parent link="${prefix}link_3"/>
       <child link="${prefix}link_4"/>

Commit message: rotation of the iiwa_base collisiion mesh by 90 about z axis

File: iiwa_description/urdf/iiwa.urdf.xacro (robot description, xacro)
@@ -8,9 +8,9 @@
   </material>
 <!-- Joint between the ${parent} and the added base -->
-  <joint name="${prefix}iiwa_root_joint" type="fixed">
-      <origin xyz = "0 0 0.86" rpy = "${PI} 0 ${-PI/2}" />
-      <parent link="${parent}"/>
-      <child link="${prefix}iiwa_base"/>
-  </joint>
+<joint name="${prefix}iiwa_root_joint" type="fixed">
+  <origin xyz = "0 0 0.86" rpy = "${PI} 0 ${-PI/2}" />
+  <parent link="${parent}"/>
+  <child link="${prefix}iiwa_base"/>
+</joint>
 <!-- Added base -->
  <link name = "${prefix}iiwa_base">
@@ -22,5 +22,5 @@
       </visual>
       <collision>
-        <origin xyz = "0 0 0" rpy = "0 0 0"/>
+        <origin xyz = "0 0 0" rpy = "0 0 ${PI/2}"/>
         <geometry>
           <mesh filename = "package://iiwa_description/meshes/flex_fellow_h800/flex_fellow_h800.stl"/>

Commit message: changed limits of joint 4

File: iiwa_description/urdf/iiwa.urdf.xacro (robot description, xacro)
@@ -242,5 +242,6 @@
       <child link="${prefix}link_4"/>
       <axis xyz="0 -1 0"/>
-      <limit effort="176" lower="-2.0942" upper="2.0942" velocity="1.3089"/>
+      <!-- <limit effort="176" lower="-2.0942" upper="2.0942" velocity="1.3089"/>  -->
+      <limit effort="176" lower="${-PI}" upper="${PI}" velocity="1.3089"/>
   </joint>
   <joint name="${prefix}joint_a5" type="revolute">

Commit message: robots neutral pose upright

File: iiwa_description/urdf/iiwa.urdf.xacro (robot description, xacro)
@@ -25,5 +25,5 @@
   </link>
   <joint name="iiwa_root_joint" type="fixed">
-    <origin xyz="-0.25 0.0 0.90" rpy="${PI} 0.0 ${PI}"/>
+    <origin xyz="-0.25 0.0 0.90" rpy="${PI} 0 ${-PI/2}"/>
     <parent link="world"/>
     <child link="iiwa_base"/>
@@ -249,5 +249,5 @@
     </joint>
     <joint name="${prefix}joint_a2" type="revolute">
-      <origin rpy="0 ${pose_dir}${PI/3} 0" xyz="-0.00043624 0 0.36"/>
+      <origin rpy="0 0 0" xyz="-0.00043624 0 0.36"/>
       <parent link="${prefix}link_1"/>
       <child link="${prefix}link_2"/>
@@ -263,5 +263,5 @@
     </joint>
     <joint name="${prefix}joint_a4" type="revolute">
-      <origin rpy="0 ${pose_dir}${PI/2} 0" xyz="0.00043624 0 0.42"/>
+      <origin rpy="0 0 0" xyz="0.00043624 0 0.42"/>
       <parent link="${prefix}link_3"/>
       <child link="${prefix}link_4"/>
@@ -277,5 +277,5 @@
     </joint>
     <joint name="${prefix}joint_a6" type="revolute">
-      <origin rpy="0 ${pose_dir}${PI/6} 0" xyz="0 0 0.4"/>
+      <origin rpy="0 0 0" xyz="0 0 0.4"/>
       <parent link="${prefix}link_5"/>
       <child link="${prefix}link_6"/>
@@ -291,5 +291,5 @@
     </joint>
     <joint name="${prefix}joint_a7-tool0" type="fixed">
-      <origin rpy="0 ${PI/2} ${PI/2}" xyz="0 -0.06 0.205"/>
+      <origin rpy="0 ${PI/2} 0" xyz="-0.05 0 0.2"/>
       <parent link="${prefix}link_7"/>
       <child link="${prefix}tool0"/>
@@ -297,5 +297,5 @@
     </joint>
     <joint name="${prefix}tcp_joint" type="fixed">
-      <origin xyz="-0.05 0.0 0.0" rpy="0.0 ${PI} 0"/>
+      <origin xyz="-0.05 0.0 0.0" rpy="0 0 0"/>
       <parent link="${prefix}tool0"/>
       <child link="${prefix}tcp"/>
